Commit message: Updated with corrections from feedback

File: my_rb1_description/urdf/my_rb1_robot.urdf (robot description, URDF)
Before this commit: robot RB1, 7 links, 6 joints
Links:
- link left_wheel: mass 0.00025 -> 0.0025
Joints:
- joint base_link_back_caster_joint: origin xyz=0.1 0.0 -0.15 rpy=0.0 0.0 0.0 -> xyz=-0.1 0.0 -0.15 rpy=0.0 0.0 0.0
- joint base_link_front_caster_joint: origin xyz=-0.1 0.0 -0.15 rpy=0.0 0.0 0.0 -> xyz=0.1 0.0 -0.15 rpy=0.0 0.0 0.0
- joint base_link_left_wheel_joint: origin xyz=0.0 0.2 -0.15 rpy=-1.5708 0.0 0.0 -> xyz=0.0 0.2 -0.15 rpy=1.5708 0.0 0.0

File: my_rb1_gazebo/urdf/my_rb1_robot_gazebo.urdf (robot description, URDF)
Before this commit: robot RB1, 7 links, 6 joints
Links:
- link left_wheel: mass 0.00025 -> 0.0025
Joints:
- joint base_link_back_caster_joint: origin xyz=0.1 0.0 -0.15 rpy=0.0 0.0 0.0 -> xyz=-0.1 0.0 -0.15 rpy=0.0 0.0 0.0
- joint base_link_front_caster_joint: origin xyz=-0.1 0.0 -0.15 rpy=0.0 0.0 0.0 -> xyz=0.1 0.0 -0.15 rpy=0.0 0.0 0.0
