Commit message: Updatd spawn launch file to include parameter bridge and fixed errors regarding urdf wheel orientation.

File: my_rb1_gazebo/urdf/my_rb1_robot_gazebo.urdf (robot description, URDF)
Before this commit: robot RB1, 7 links, 6 joints
Joints:
- joint base_link_right_wheel_joint: origin xyz=0.0 -0.2 -0.15 rpy=1.5708 0.0 0.0 -> xyz=0.0 -0.2 -0.15 rpy=-1.5708 0.0 0.0

Commit message: Package migration from Gazebo Sim to Classice

File: my_rb1_gazebo/urdf/my_rb1_robot_gazebo.urdf (robot description, URDF)
Before this commit: robot RB1, 7 links, 6 joints
Links:
- link back_caster: mass 0.02747 -> 0.5
- link base_link: mass 24.72479 -> 20.5
- link front_caster: mass 0.02747 -> 0.5
- link front_laser: mass 0.21977 -> None; geometry 
- link left_wheel: mass 0.0025 -> 1.5
- link right_wheel: mass 0.0025 -> 1.5
Joints:
- joint base_link_back_caster_joint: origin xyz=-0.1 0.0 -0.15 rpy=0.0 0.0 0.0 -> xyz=-0.1 0.0 -0.15 rpy=0 0 0
- joint base_link_front_caster_joint: origin xyz=0.1 0.0 -0.15 rpy=0.0 0.0 0.0 -> xyz=0.1 0.0 -0.15 rpy=0 0 0
- joint base_link_front_laser_joint: origin xyz=0.25 0.0 0.075 rpy=3.14159 0.0 0.0 -> xyz=0.25 0 0.075 rpy=3.14 0 0
- joint base_link_left_wheel_joint: axis 0 0 1 -> 0 1 0; origin xyz=0.0 0.2 -0.15 rpy=-1.5708 0.0 0.0 -> xyz=0 0.2 -0.15 rpy=0 0 0
- joint base_link_plate_joint: child base_footprint -> base_link; origin xyz=0.0 0.0 -0.15 rpy=0.0 0.0 0.0 -> xyz=0 0 0.15 rpy=0 0 0; parent base_link -> base_footprint
- joint base_link_right_wheel_joint: axis 0 0 1 -> 0 1 0; origin xyz=0.0 -0.2 -0.15 rpy=-1.5708 0.0 0.0 -> xyz=0 -0.2 -0.15 rpy=0 0 0
